File: SingleKey_ESP32-c3/SingleKey_ESP32-c3.kicad_pcb (KiCad board)
At the start: 4 copper layers, 19 x 31 mm, 16 parts, among them J1 USB_A, SW1 SW_Push, SW3 SW_Push, U1 ESP32-C3FH4, U2 LM1117-3.3, Y1 Crystal_GND24

Commit message: PCBtweaks
Other:
- board text added: "Adam Anderson 2022"
- board text added: "BADBOARDS"
- board text added: "SINGLEKEY"
Changed lines of the file:
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@@
   (gr_line (start 86.555 70.5) (end 86.555 89.5) (layer "Edge.Cuts") (width 0.1))
   (gr_line (start 86.555 89.5) (end 90.055 89.5) (layer "Edge.Cuts") (width 0.1))
+  (gr_text "BADBOARDS" (at 88 80 270) (layer "B.SilkS")
+    (effects (font (size 2 2) (thickness 0.3) italic) (justify mirror))
+  )
+  (gr_text "SINGLEKEY" (at 104 80 90) (layer "B.SilkS")
+    (effects (font (size 2 2) (thickness 0.3) italic) (justify mirror))
+  )
+  (gr_text "Adam Anderson 2022" (at 96 72) (layer "F.SilkS")
+    (effects (font (size 1 1) (thickness 0.15)))
+  )
   (segment (start 98.75 89.5) (end 99.575 88.675) (width 0.5) (layer "F.Cu") (net 1))
   (segment (start 101.25 85.275) (end 101.275 85.275) (width 0.25) (layer "F.Cu") (net 1))
